Commit message: updated-for-ouster

File: ouster_description/urdf/OS1-64.urdf.xacro (robot description, xacro)
@@ -2,5 +2,5 @@
 <robot xmlns:xacro="http://www.ros.org/wiki/xacro" name="OS1-64">
   <xacro:property name="M_PI" value="3.1415926535897931" />
-  <xacro:macro name="OS1-64" params="*origin parent:=base_link name:=ouster topic_points:=/ouster/points topic_imu:=/ouster/imu hz:=10 lasers:=64 samples:=512 min_range:=0.9 max_range:=75.0 noise:=0.008 min_angle:=-${M_PI} max_angle:=${M_PI} organize_cloud:=true lidar_link:=ouster_lidar imu_link:=ouster_imu vfov_min:=-.26 vfov_max:=.26">
+  <xacro:macro name="OS1-64" params="*origin parent:=base_link name:=ouster topic:=/ouster/points topic_imu:=/ouster/imu hz:=10 lasers:=64 samples:=512 gpu:=false min_range:=0.9 max_range:=75.0 noise:=0.008 min_angle:=-${M_PI} max_angle:=${M_PI} organize_cloud:=true lidar_link:=ouster_lidar imu_link:=ouster_imu vfov_min:=-.26 vfov_max:=.26">
     <joint name="${name}_base_mount_joint" type="fixed">
       <xacro:insert_block name="origin" />
@@ -71,5 +71,5 @@
           </ray>
           <plugin name="gazebo_ros_laser_controller" filename="libgazebo_ros_ouster_laser.so">
-            <topicName>${topic_points}</topicName>
+            <topicName>${topic}</topicName>
             <frameName>${lidar_link}</frameName>
             <organize_cloud>${organize_cloud}</organize_cloud>
